Commit message: attach camera to robot and display the robot in gazebo

File: ob1_base_description/urdf/drivetrain.urdf.xacro (robot description, xacro)
@@ -2,4 +2,6 @@
 <robot name="drivetrain" xmlns:xacro="http://ros.org/wiki/xacro">
   <xacro:include filename="$(find ob1_base_description)/urdf/drivetrain_specs/drivetrain_specs.urdf"/>
+  <xacro:include filename="$(find ob1_base_description)/urdf/ob1_base.gazebo.xacro"/>
+  <xacro:include filename="$(find realsense2_description)/urdf/_d435.urdf.xacro" />
   <link name="base_footprint"/>
   <joint name="base_joint" type="fixed">
@@ -8,3 +10,12 @@
     <origin xyz="0.0 0.0 0.010" rpy="0 0 0"/>
   </joint>
+  <link name="base_scan"/>
+  <xacro:sensor_d435 name="camera" topics_ns="camera" parent="base_scan" publish_pointcloud="true">
+    <origin xyz="0 0 0" rpy="1.57079632679 -1.57079632679 0" />
+  </xacro:sensor_d435>
+  <joint name="scan_joint" type="fixed">
+    <parent link="base_link"/>
+    <child link="base_scan"/>
+    <origin xyz="0.275 0 0.41" rpy="1.57 0 1.57"/>
+  </joint>
 </robot>

File: ob1_base_description/urdf/drivetrain_specs/drivetrain_specs.urdf (robot description, URDF)
Before this commit: robot drivetrain_specs, 5 links, 4 joints
Links:
- removed link wheel_link
- removed link wheel_link_2
- added link wheel_left_link, mass 0; collision mesh filename=package://ob1_base_description/urdf/drivetrain_specs/wheel_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; visual mesh filename=package://ob1_base_description/urdf/drivetrain_specs/wheel_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
- added link wheel_right_link, mass 0; collision mesh filename=package://ob1_base_description/urdf/drivetrain_specs/wheel_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; visual mesh filename=package://ob1_base_description/urdf/drivetrain_specs/wheel_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
Joints:
- joint left_wheel_joint_and_base_joint: child wheel_link -> wheel_left_link
- joint right_wheel_and_base_joint: child wheel_link_2 -> wheel_right_link

File: ob1_base_description/urdf/ob1_base.gazebo.xacro (robot description, xacro)
@@ -48,6 +48,6 @@
       <legacyMode>false</legacyMode>
       <updateRate>30</updateRate>
-      <leftJoint>wheel_left_joint</leftJoint>
-      <rightJoint>wheel_right_joint</rightJoint>
+      <leftJoint>left_wheel_joint_and_base_joint</leftJoint>
+      <rightJoint>right_wheel_joint_and_base_joint</rightJoint>
       <wheelSeparation>0.287</wheelSeparation>
       <wheelDiameter>0.066</wheelDiameter>

Commit message: attach camera at the front of robot

File: ob1_base_description/urdf/drivetrain.urdf.xacro (robot description, xacro)
@@ -17,5 +17,6 @@
     <parent link="base_link"/>
     <child link="base_scan"/>
-    <origin xyz="0.275 0 0.41" rpy="1.57 0 1.57"/>
+    <!-- <origin xyz="0.275 0 0.41" rpy="1.57 0 1.57"/> -->
+    <origin xyz="0 -0.275 0.41" rpy="1.57 0 0"/>
   </joint>
 </robot>
