Commit message: download missing parts and automatically define joints

File: ob1_base_description/urdf/drivetrain_specs/drivetrain_specs.urdf (robot description, URDF)
Before this commit: robot drivetrain_specs, 1 links, 0 joints
Links:
- added link caster_link, mass 0; collision mesh filename=package://ob1_base_description/urdf/drivetrain_specs/caster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; visual mesh filename=package://ob1_base_description/urdf/drivetrain_specs/caster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
- added link torso_link, mass 0; collision mesh filename=package://ob1_base_description/urdf/drivetrain_specs/1ft_30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; collision mesh filename=package://ob1_base_description/urdf/drivetrain_specs/1ft_30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
- added link wheel_link, mass 0; collision mesh filename=package://ob1_base_description/urdf/drivetrain_specs/wheel_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; visual mesh filename=package://ob1_base_description/urdf/drivetrain_specsob1_bas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
- added link wheel_link_2, mass 0; collision mesh filename=package://ob1_base_description/urdf/drivetrain_specs/wheel_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; visual mesh filename=package://ob1_base_description/urdf/drivetrain_specs/wheel_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
- link base_link: geometry collision mesh filename=package://ob1_base_description/urdf/drivetrain_specs/217-25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; collision mesh filename=package://ob1_base_description/urdf/drivetrain_specs/217-25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
Joints:
- added joint caster_and_base_joint: type continuous, parent base_link, child caster_link, origin xyz=-0.30003749967508885899 -0.028466248845019893887 -0.26454124870035566897 rpy=-3.2558828317096316961e-64 -1.4663192707649492644e-48 3.141592653589793116, axis 0 0 1, limit effort=1 velocity=20
- added joint left_wheel_joint_and_base_joint: type continuous, parent base_link, child wheel_link_2, origin xyz=6.498223625861498931e-10 0 -0.5614449987003558018 rpy=1.9366355108736570128e-16 7.395570986446984581e-32 0, axis 0 0 1, limit effort=1 velocity=20
- added joint right_wheel_and_base_joint: type continuous, parent base_link, child wheel_link, origin xyz=0.28048014598486692428 0.1321445608618717904 -0.060433751154980112907 rpy=1.570796326794896558 -0 1.570796326794896558, axis 0 0 1, limit effort=1 velocity=20
- added joint torso_and_base_joint: type fixed, parent base_link, child torso_link, origin xyz=-0.067000059675029949302 0.43158375162706152928 -0.2804926086147819797 rpy=-1.57079632679489678 5.7144181737427606316e-15 -3.141592653589793116, axis 0 0 1, limit effort=1 velocity=20

Commit message: fix the order of right wheel and base joint

File: ob1_base_description/urdf/drivetrain_specs/drivetrain_specs.urdf (robot description, URDF)
Before this commit: robot drivetrain_specs, 5 links, 4 joints
Links:
- link wheel_link: geometry collision mesh filename=package://ob1_base_description/urdf/drivetrain_specs/wheel_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; visual mesh filename=package://ob1_base_description/urdf/drivetrain_specs/wheel_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
Joints:
- joint caster_and_base_joint: origin xyz=-0.30003749967508885899 -0.028466248845019893887 -0.26454124870035566897 rpy=-3.2558828317096316961e-64 -1.4663192707649492644e-48 3.141592653589793116 -> xyz=0.015938897284511241437 -0.16789293881321706858 -0.088900000000000006795 rpy=-1.570796326794896558 -2.2204460492503135739e-16 -1.570796326794896558
- joint left_wheel_joint_and_base_joint: child wheel_link_2 -> wheel_link; origin xyz=6.498223625861498931e-10 0 -0.5614449987003558018 rpy=1.9366355108736570128e-16 7.395570986446984581e-32 0 -> xyz=-0.28096485271548882201 0.13214456151169415299 -0.060433751154980112907 rpy=1.57079632679489678 -0 1.570796326794896558
- joint right_wheel_and_base_joint: child wheel_link -> wheel_link_2; origin xyz=0.28048014598486692428 0.1321445608618717904 -0.060433751154980112907 rpy=1.570796326794896558 -0 1.570796326794896558 -> xyz=0.28048014598486692428 0.1321445608618717904 -0.060433751154980119846 rpy=-1.570796326794896558 -0 1.570796326794896558
- joint torso_and_base_joint: origin xyz=-0.067000059675029949302 0.43158375162706152928 -0.2804926086147819797 rpy=-1.57079632679489678 5.7144181737427606316e-15 -3.141592653589793116 -> xyz=-1.2462629915069300957e-05 0.065144501186841841101 0.37115000047208140943 rpy=3.141592653589793116 1.156482317317871725e-16 -1.5707963267949023312

Commit message: rename the link for more consisentcy

File: ob1_base_description/urdf/drivetrain_specs/drivetrain_specs.urdf (robot description, URDF)
Before this commit: robot drivetrain_specs, 5 links, 4 joints
Joints:
- removed joint left_wheel_joint_and_base_joint
- added joint left_wheel_and_base_joint: type continuous, parent base_link, child wheel_left_link, origin xyz=-0.28096485271548882201 0.13214456151169415299 -0.060433751154980112907 rpy=1.57079632679489678 -0 1.570796326794896558, axis 0 0 1, limit effort=1 velocity=20

File: ob1_base_description/urdf/ob1_base.gazebo.xacro (robot description, xacro)
@@ -48,6 +48,6 @@
       <legacyMode>false</legacyMode>
       <updateRate>30</updateRate>
-      <leftJoint>left_wheel_joint_and_base_joint</leftJoint>
-      <rightJoint>right_wheel_joint_and_base_joint</rightJoint>
+      <leftJoint>left_wheel_and_base_joint</leftJoint>
+      <rightJoint>right_wheel_and_base_joint</rightJoint>
       <wheelSeparation>0.287</wheelSeparation>
       <wheelDiameter>0.066</wheelDiameter>

Commit message: add inertia to wheels

File: ob1_base_description/urdf/drivetrain_specs/drivetrain_specs.urdf (robot description, URDF)
Before this commit: robot drivetrain_specs, 5 links, 4 joints
Links:
- link caster_link: mass 0 -> 0.005
- link wheel_left_link: mass 0 -> 2.8498940e-02
- link wheel_right_link: mass 0 -> 2.8498940e-02

Commit message: remove floating points

File: ob1_base_description/urdf/drivetrain_specs/drivetrain_specs.urdf (robot description, URDF)
Before this commit: robot drivetrain_specs, 5 links, 4 joints
Links:
- link base_link: geometry collision mesh filename=package://ob1_base_description/urdf/drivetrain_specs/217-25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; collision mesh filename=package://ob1_base_description/urdf/drivetrain_specs/217-25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

Commit message: Fix URDF and Gazebo Bugs (#10)
* attach camera at the front of robot

* attach camera at the front of robot

* add inertia to wheels

* remove floating points

File: ob1_base_description/urdf/drivetrain_specs/drivetrain_specs.urdf (robot description, URDF)
Before this commit: robot drivetrain_specs, 5 links, 4 joints
Links:
- link base_link: geometry collision mesh filename=package://ob1_base_description/urdf/drivetrain_specs/217-25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; collision mesh filename=package://ob1_base_description/urdf/drivetrain_specs/217-25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
- link caster_link: mass 0 -> 0.005
- link wheel_left_link: mass 0 -> 2.8498940e-02
- link wheel_right_link: mass 0 -> 2.8498940e-02
